File: kicad/elv-usb-i2c-adapter.sch (KiCad schematic (older format))
At the start: 8 parts, among them IC1 ATmega88PA-AU, IC2 CP2102N-A01-GQFN24, IC3 74HC14

Commit message: Creating a schematic
Parts:
- removed IC2: CP2102N-A01-GQFN24, Package_DFN_QFN:QFN-24-1EP_4x4mm_P0.5mm_EP2.6x2.6mm, symbol Interface_USB:CP2102N-A01-GQFN24
- added C3: C_Small, symbol Device:C_Small
- added D1: LED, symbol Device:LED
- added R2, R3, R6: 10k, symbol Device:R
- added R4: 4k7, symbol Device:R
- added RG1: R, symbol Device:R
Connections:
- net labels added: +5V, ACT, DM, DP, GND, MISO, MOSI, RESET, RST, RX, RXD, SCK, SCL, SDA, SS, SUSPEND, TX, TXD, VBUS
- wire segments 0 -> 62
- no-connect marks 0 -> 19
Other:
- moved on the sheet: BU1, IC1, IC3G, PRG1, ST1, ST2, ST3
